File: Kicad/Remotino Nano Dual Rail/Remotino Nano2.kicad_sch (KiCad schematic)
At the start: 27 parts, among them J1 Conn_01x15_Socket, J10 I2C_ESPANSIONE, J11 Conn_01x06_Socket, J12 Conn_01x06_Socket, J13 ALIM_12V, J15 Conn_01x01_Pin, J16 Conn_01x01_Pin, J17 Conn_01x01_Pin, J2 Conn_01x15_Socket, J3 Conn_01x06_Socket, J4 Conn_02x05_SCHEDA-8-RELE-SCAM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, J5 Conn_01x02_Pin, J6 Conn_01x02_Pin, J7 BINARIO2, J8 BINARIO1, J9 ALIM_12V, Q1 BC337, Q2 BC337, U1 TSOP23xx

Commit message: aggiornamenti
Parts:
- added RV1, RV2: 10k, symbol Device:R_Potentiometer_Trim
Connections:
- net +5NANO: now also RV1.1, RV2.1
- net 0: now also RV1.3, RV2.3
- net at J1.5 (Pin_5): now also RV1.2
- net at J1.6 (Pin_6): now also RV2.2
- no-connect marks 11 -> 9

Commit message: aggiunto potenziometri
aggiunto potenz.
Parts:
- removed RV1, RV2: 10k, symbol Device:R_Potentiometer_Trim
- added RV3, RV4, RV5, RV6, RV7: 10k, symbol Device:R_Potentiometer_Trim
- J13: value ALIM_12V -> ALIM_5V
Connections:
- net +5NANO: now also RV3.1, RV4.1, RV5.1, RV6.1, RV7.1
- net 0: now also RV3.3, RV4.3, RV5.3, RV6.3, RV7.3
- net at J1.10 (Pin_10): now also RV6.2
- net at J1.11 (Pin_11): now also RV7.2
- net at J1.5 (Pin_5): now also RV3.2
- net at J1.6 (Pin_6): now also RV4.2
- net at J1.7 (Pin_7): now also RV5.2
- no-connect marks 9 -> 6
Other:
- note added: "Potenziometri o trimmer 1 valore boost 2 valore minimum speed 3 accelerazione 4 decelerazione 5 deceleraz. fermata automatica"
- moved on the sheet: J13
